Commit message: plus altra

File: g7_openarm/g7_openarm_description/urdf/g7_openarm.urdf (robot description, URDF)
Before this commit: robot g7_openarm, 31 links, 30 joints
Joints:
- joint L_ee_joint: origin xyz=0 -0.03175 -0.119 rpy=0 0 0 -> xyz=0 -0.03175 -0.135 rpy=0 0 0
- joint R_ee_joint: origin xyz=0 0.03175 -0.119 rpy=0 0 0 -> xyz=0 0.03175 -0.135 rpy=0 0 0
